Commit message: added IMU joint, fixed inverse_kinematics, created new URDF

File: werdna_description/urdf/consts.xacro (robot description, xacro)
@@ -18,3 +18,34 @@
     <xacro:property name="wheel_radius" value="0.0855"/>
     <xacro:property name="wheel_lenght" value="0.045"/>
+    <material name="white">
+        <color rgba="1 1 1 1" />
+    </material>
+    <material name="orange">
+        <color rgba="1 0.3 0.1 1"/>
+    </material>
+    <material name="blue">
+        <color rgba="0.2 0.2 1 1"/>
+    </material>
+    <material name="black">
+        <color rgba="0 0 0 1"/>
+    </material>
+    <material name="red">
+        <color rgba="1 0 0 1"/>
+    </material>
+    <xacro:property name="wheel_radius" value="0.0855"/>
+    <xacro:property name="wheel_length" value="0.045"/>
+    <!-- Width, length, height = x,y,z -->
+    <xacro:property name="chassis_length" value="0.2"/>
+    <xacro:property name="chassis_width" value="0.15"/>
+    <xacro:property name="chassis_height" value="0.12"/>
+    <xacro:property name="imu_length" value="0.01"/>
+    <xacro:property name="imu_width" value="0.01"/>
+    <xacro:property name="imu_height" value="0.01"/>
+    <xacro:property name="rod_length" value="0.05"/>
+    <xacro:property name="rod_width" value="0.05"/>
+    <xacro:property name="rod_height" value="0.2"/>
+    <xacro:property name="chassis_mass" value="2.0"/>
+    <xacro:property name="rod_mass" value="1.0"/>
+    <xacro:property name="wheel_mass" value="2.2"/>
+    <xacro:property name="imu_mass" value="0.01"/>
 </robot>

File: werdna_description/urdf/ros2_control.xacro (robot description, xacro)
@@ -56,5 +56,5 @@
     <gazebo>
         <plugin name="gazebo_ros2_control" filename="libgazebo_ros2_control.so">
-            <parameters>$(find werdna_description)/config/werdna_joint_controller.yaml</parameters>
+            <parameters>$(find bringup)/configs/ros2_controllers.yaml</parameters>
         </plugin>
     </gazebo>

File: werdna_description/urdf/werdna_core.xacro (robot description, xacro)
@@ -1,10 +1,6 @@
 <?xml version="1.0"?>
 <robot name='werdna' xmlns:xacro="http://www.ros.org/wiki/xacro">
-    <!-- links -->
-    <xacro:include filename='werdna_links.xacro'/>
-    <!-- joints -->
-    <xacro:include filename="werdna_joints.xacro"/>
-    <!-- Others -->
+    <xacro:include filename='werdna.xacro'/>
+    <xacro:include filename="werdna_gazebo.xacro"/>
     <xacro:include filename="ros2_control.xacro"/>
-    <xacro:include filename="werdna_gazebo.xacro"/>
 </robot>

File: werdna_description/urdf/werdna_gazebo.xacro (robot description, xacro)
@@ -1,57 +1,91 @@
-<?xml version="1.0"?>
-<robot xmlns:xacro="http://www.ros.org/wiki/xacro">
-    <xacro:include filename:'physics.xacro'/>
-    <xacro:macro name='hip'>
-        <mu1>0.2</mu1>
-        <mu2>0.2</mu2>
-        <maxVel>0.01</maxVel>
-        <self_collide>1</self_collide>
-        <material>Gazebo/Red</material>
-    <xacro:macro>
-    <xacro:macro name='knee'>
-        <mu1>0.2</mu1>
-        <mu2>0.2</mu2>
-        <maxVel>0.01</maxVel>
-        <self_collide>1</self_collide>
-        <material>Gazebo/Orange</material>
-    <xacro:macro>
-    <xacro:macro name='wheel'>
-        <mu1>0.9</mu1>
-        <mu2>0.9</mu2>
-        <fdir1>1 0 0</fdir1>
-        <maxVel>0.0</maxVel>
-        <maxContacts>1</maxContacts>
-        <gravity>true</gravity>
-        <restitution_coefficient>1</restitution_coefficient>
-        <threshold>0</threshold>
-        <self_collide>1</self_collide>
-        <material>Gazebo/Black</material>
-    <xacro:macro>
-    <!-- body  -->
-    <gazebo reference="base_link">
-        <mu1>0.05</mu1>
-        <mu2>0.05</mu2>
-        <maxVel>0.01</maxVel>
-        <material>Gazebo/DarkGrey</material>
-    </gazebo>
-    <!-- hip -->
-    <gazebo reference="left_hip_link">
-        <xacro:hip></xacro:hip>
-    </gazebo>
-    <gazebo reference="right_hip_link">
-        <xacro:hip></xacro:hip>
-    </gazebo>
-    <!-- knee -->
-    <gazebo reference="left_knee_link">
-        <xacro:knee></xacro:knee>
-    </gazebo>
-    <gazebo reference="right_knee_link">
-        <xacro:knee></xacro:knee>
-    </gazebo>
-    <gazebo reference="left_wheel_link">
-        <xacro:wheel></xacro:wheel>
-    </gazebo>
-    <gazebo reference="right_hip_link">
-        <xacro:wheel></xacro:wheel>
-    </gazebo>
+<?xml version="1.0" ?>
+<robot name="Model_URDF" xmlns:xacro="http://www.ros.org/wiki/xacro" >
+<gazebo reference="chassis_link">
+  <material>Gazebo/Blue</material>
+  <mu1>0.2</mu1>
+  <mu2>0.2</mu2>
+  <self_collide>true</self_collide>
+  <gravity>true</gravity>
+</gazebo>
+<gazebo reference="imu_link">
+  <material>Gazebo/White</material>
+  <mu1>0.2</mu1>
+  <mu2>0.2</mu2>
+  <self_collide>true</self_collide>
+  <gravity>true</gravity>
+</gazebo>
+<gazebo reference="left_hip_link">
+  <material>Gazebo/Orange</material>
+  <mu1>0.2</mu1>
+  <mu2>0.2</mu2>
+  <maxVel>0.01</maxVel>
+  <self_collide>true</self_collide>
+</gazebo>
+<gazebo reference="left_knee_link">
+  <material>Gazebo/Red</material>
+  <mu1>0.2</mu1>
+  <mu2>0.2</mu2>
+  <maxVel>0.01</maxVel>
+  <self_collide>true</self_collide>
+</gazebo>
+<gazebo reference="left_wheel">
+  <mu1>0.9</mu1>
+  <mu2>0.9</mu2>
+  <fdir1>1 0 0</fdir1>
+  <maxVel>0.0</maxVel>
+  <maxContacts>1</maxContacts>
+  <gravity>true</gravity>
+  <restitution_coefficient>1</restitution_coefficient>
+  <threshold>0</threshold>
+  <self_collide>1</self_collide>
+  <material>Gazebo/Black</material>
+</gazebo>
+<gazebo reference="right_hip_link">
+  <material>Gazebo/Orange</material>
+  <mu1>0.2</mu1>
+  <mu2>0.2</mu2>
+  <maxVel>0.01</maxVel>
+  <self_collide>true</self_collide>
+</gazebo>
+<gazebo reference="right_knee_link">
+  <material>Gazebo/Red</material>
+  <mu1>0.2</mu1>
+  <mu2>0.2</mu2>
+  <maxVel>0.01</maxVel>
+  <self_collide>true</self_collide>
+</gazebo>
+<gazebo reference="right_wheel">
+  <mu1>0.9</mu1>
+  <mu2>0.9</mu2>
+  <fdir1>1 0 0</fdir1>
+  <maxVel>0.0</maxVel>
+  <maxContacts>1</maxContacts>
+  <gravity>true</gravity>
+  <restitution_coefficient>1</restitution_coefficient>
+  <threshold>0</threshold>
+  <self_collide>1</self_collide>
+  <material>Gazebo/Black</material>
+</gazebo>
+<gazebo reference="imu_link">
+  <sensor name="imu_sensor" type="imu">
+    <always_on>true</always_on>
+    <update_rate>100</update_rate>
+    <visualize>true</visualize>
+    <topic>__default_topic__</topic>
+    <plugin filename="libgazebo_ros_imu_sensor.so" name="imu_plugin">
+      <topicName>imu</topicName> <!-- Ensure this matches your UKF config -->
+      <bodyName>imu_link</bodyName>   <!-- This should be the same as the IMU link name -->
+      <updateRateHZ>100.0</updateRateHZ>
+      <gaussianNoise>0.0</gaussianNoise>
+      <xyzOffset>0 0 0</xyzOffset>
+      <rpyOffset>0 0 0</rpyOffset>
+      <frameName>imu</frameName> <!-- Frame name for TF broadcasts -->
+      <ros>
+        <remapping>~/out:=/imu</remapping> <!-- ROS 2 topic remapping -->
+      </ros>
+      <initialOrientationAsReference>false</initialOrientationAsReference>
+    </plugin>
+    <pose>0 0 0 0 0 0</pose>
+  </sensor>
+</gazebo>
 </robot>

Commit message: Update

File: werdna_description/urdf/consts.xacro (robot description, xacro)
@@ -2,17 +2,17 @@
 <robot xmlns:xacro="http://www.ros.org/wiki/xacro">
     <!-- joint's limits -->
-    <xacro:property name="hip_high_limit" value="1.047198"/>
-    <xacro:property name="hip_low_limit" value="-1.047198"/>
-    <xacro:property name="knee_high_limit" value="2.094395"/>
-    <xacro:property name="knee_low_limit" value="-2.094395"/>
-    <xacro:property name="velocity" value="1"/>
-    <xacro:property name="effort" value="10"/>
+    <xacro:property name="hip_high_limit" value="3.142"/>
+    <xacro:property name="hip_low_limit" value="-3.142"/>
+    <xacro:property name="knee_high_limit" value="3.142"/>
+    <xacro:property name="knee_low_limit" value="-3.142"/>
+    <xacro:property name="velocity" value="100.0"/>
+    <xacro:property name="effort" value="10.0"/>
     <!-- joint's dynamics -->
     <xacro:property name="use_dynamics" value="true"/>
     <xacro:macro name="hip_joint_dynamics">
-        <dynamics damping="0.01" friction="10000"/>
+        <dynamics friction="2000"/>
     </xacro:macro>
     <xacro:macro name="knee_joint_dynamics">
-        <dynamics damping="0.01" friction="10000"/>
+        <dynamics friction="2000"/>
     </xacro:macro>
     <xacro:property name="wheel_radius" value="0.0855"/>
@@ -45,5 +45,5 @@
     <xacro:property name="rod_width" value="0.05"/>
     <xacro:property name="rod_height" value="0.2"/>
-    <xacro:property name="chassis_mass" value="2.0"/>
+    <xacro:property name="chassis_mass" value="4.0"/>
     <xacro:property name="rod_mass" value="1.0"/>
     <xacro:property name="wheel_mass" value="2.2"/>

File: werdna_description/urdf/ros2_control_sim.xacro (robot description, xacro)
@@ -7,6 +7,6 @@
         <joint name="left_hip_joint">
             <command_interface name="position">
-                <param name="min">-1.047198</param>
-                <param name="max">1.047198</param>
+                <param name="min">-3.142</param>
+                <param name="max">3.142</param>
             </command_interface>
             <state_interface name="position"/>
@@ -15,6 +15,6 @@
         <joint name="left_knee_joint">
             <command_interface name="position">
-                <param name="min">-1.047198</param>
-                <param name="max">2.094395</param>
+                <param name="min">-3.142</param>
+                <param name="max">3.142</param>
             </command_interface>
             <state_interface name="position"/>
@@ -23,17 +23,17 @@
         <joint name="right_hip_joint">
             <command_interface name="position">
-                <param name="min">-1.047198</param>
-                <param name="max">1.047198</param>
+                <param name="min">-3.142</param>
+                <param name="max">3.142</param>
             </command_interface>
+            <state_interface name="position"/>
             <state_interface name="velocity"/>
-            <state_interface name="position"/>
         </joint>
         <joint name="right_knee_joint">
             <command_interface name="position">
-                <param name="min">-2.094395</param>
-                <param name="max">1.047198</param>
+                <param name="min">-3.142</param>
+                <param name="max">3.142</param>
             </command_interface>
+            <state_interface name="position"/>
             <state_interface name="velocity"/>
-            <state_interface name="position"/>
         </joint>
         <joint name="left_wheel_joint">

File: werdna_description/urdf/werdna_core.xacro (robot description, xacro)
@@ -3,4 +3,4 @@
     <xacro:include filename='werdna.xacro'/>
     <xacro:include filename="werdna_gazebo.xacro"/>
-    <xacro:include filename="ros2_control.xacro"/>
+    <xacro:include filename="ros2_control_sim.xacro"/>
 </robot>

File: werdna_description/urdf/werdna_gazebo.xacro (robot description, xacro)
@@ -2,7 +2,7 @@
 <robot name="Model_URDF" xmlns:xacro="http://www.ros.org/wiki/xacro" >
 <gazebo reference="chassis_link">
-  <material>Gazebo/Blue</material>
   <mu1>0.2</mu1>
   <mu2>0.2</mu2>
+  <material>Gazebo/Blue</material>
   <self_collide>true</self_collide>
   <gravity>true</gravity>
@@ -10,6 +10,4 @@
 <gazebo reference="imu_link">
   <material>Gazebo/White</material>
-  <mu1>0.2</mu1>
-  <mu2>0.2</mu2>
   <self_collide>true</self_collide>
   <gravity>true</gravity>
@@ -17,25 +15,17 @@
 <gazebo reference="left_hip_link">
   <material>Gazebo/Orange</material>
-  <mu1>0.2</mu1>
-  <mu2>0.2</mu2>
   <maxVel>0.01</maxVel>
-  <self_collide>true</self_collide>
+  <!-- <self_collide>true</self_collide> -->
 </gazebo>
 <gazebo reference="left_knee_link">
   <material>Gazebo/Red</material>
-  <mu1>0.2</mu1>
-  <mu2>0.2</mu2>
   <maxVel>0.01</maxVel>
-  <self_collide>true</self_collide>
+  <!-- <self_collide>true</self_collide> -->
 </gazebo>
 <gazebo reference="left_wheel">
-  <mu1>0.9</mu1>
-  <mu2>0.9</mu2>
-  <fdir1>1 0 0</fdir1>
-  <maxVel>0.0</maxVel>
+  <mu1>0.5</mu1>
+  <mu2>0.5</mu2>
   <maxContacts>1</maxContacts>
   <gravity>true</gravity>
-  <restitution_coefficient>1</restitution_coefficient>
-  <threshold>0</threshold>
   <self_collide>1</self_collide>
   <material>Gazebo/Black</material>
@@ -43,25 +33,17 @@
 <gazebo reference="right_hip_link">
   <material>Gazebo/Orange</material>
-  <mu1>0.2</mu1>
-  <mu2>0.2</mu2>
   <maxVel>0.01</maxVel>
-  <self_collide>true</self_collide>
+  <!-- <self_collide>true</self_collide> -->
 </gazebo>
 <gazebo reference="right_knee_link">
   <material>Gazebo/Red</material>
-  <mu1>0.2</mu1>
-  <mu2>0.2</mu2>
   <maxVel>0.01</maxVel>
-  <self_collide>true</self_collide>
+  <!-- <self_collide>true</self_collide> -->
 </gazebo>
 <gazebo reference="right_wheel">
-  <mu1>0.9</mu1>
-  <mu2>0.9</mu2>
-  <fdir1>1 0 0</fdir1>
-  <maxVel>0.0</maxVel>
+  <mu1>0.5</mu1>
+  <mu2>0.5</mu2>
   <maxContacts>1</maxContacts>
   <gravity>true</gravity>
-  <restitution_coefficient>1</restitution_coefficient>
-  <threshold>0</threshold>
   <self_collide>1</self_collide>
   <material>Gazebo/Black</material>

File: werdna_description/werdna.xacro (robot description, xacro)
@@ -1,6 +1,6 @@
 <?xml version="1.0"?>
 <robot name='werdna' xmlns:xacro="http://www.ros.org/wiki/xacro">
-    <xacro:include filename="consts.xacro"/>
-    <xacro:include filename='inertial_macros.xacro'/>
+    <xacro:include filename="urdf/consts.xacro"/>
+    <xacro:include filename='urdf/inertial_macros.xacro'/>
     <!-- Limits -->
     <xacro:macro name="hip_limits">
@@ -11,6 +11,5 @@
     </xacro:macro>
     <!-- *********** base link *********** -->
-    <link name="base_link"></link>
-    <link name="chassis_link">
+    <link name="base_link">
         <xacro:inertial_box mass="${chassis_mass}" x="${chassis_length}" y="${chassis_width}" z="${chassis_height}">
             <origin xyz="0 0 0" rpy="0 0 0"/>
@@ -29,22 +28,4 @@
             </geometry>
             <material name="blue"/>
-        </collision>
-    </link>
-    <link name="castor_link">
-        <xacro:inertial_sphere mass="${0.02}" radius="0.01725">
-            <origin xyz="0 0 0" rpy="0 0 0"/>
-        </xacro:inertial_sphere>
-        <visual>
-            <origin xyz="0.0 0.0 0.0" rpy="0.0 0.0 0.0"/>
-            <geometry>
-                <sphere radius="0.01725"/>
-            </geometry>
-            <material name="white"/>
-        </visual>
-        <collision>
-            <origin xyz="0.0 0.0 0.0" rpy="0.0 0.0 0.0"/>
-            <geometry>
-                <sphere radius="0.01725"/>
-            </geometry>
         </collision>
     </link>
@@ -184,25 +165,14 @@
         </xacro:inertial_cylinder>
     </link>
-    <!-- chassis_joint -->
-    <joint name="chassis_joint" type="fixed">
-        <origin xyz="0.0 0.0 ${chassis_height/2}" rpy="0.0 0.0 0.0"/>
-        <parent link="base_link"/>
-        <child link="chassis_link"/>
-    </joint>
     <!-- imu joint -->
     <joint name="imu_joint" type="fixed">
         <origin xyz="0.0 0.0 ${chassis_height/2 + imu_height/2}" rpy="0.0 0.0 0.0"/>
-        <parent link="chassis_link"/>
+        <parent link="base_link"/>
         <child link="imu_link"/>
-    </joint>
-    <joint name="castor_joint" type="fixed">
-        <origin xyz="0.0 0.0 -${chassis_height/2}" rpy="0.0 0.0 0.0"/>
-        <parent link="chassis_link"/>
-        <child link="castor_link"/>
     </joint>
     <!-- hip joints -->
     <joint name="left_hip_joint" type="revolute">
         <origin xyz="0.0 ${chassis_width/2 + rod_width/2} 0.0" rpy="0.0 ${3.142/2} 0.0"/>
-        <parent link="chassis_link"/>
+        <parent link="base_link"/>
         <child link="left_hip_link"/>
         <axis xyz="0.0 1.0 0.0"/>
@@ -214,5 +184,5 @@
     <joint name="right_hip_joint" type="revolute">
         <origin xyz="0.0 -${chassis_width/2 + rod_width/2} 0.0" rpy="0.0 ${3.142/2} 0.0"/>
-        <parent link="chassis_link"/>
+        <parent link="base_link"/>
         <child link="right_hip_link"/>
         <axis xyz="0.0 1.0 0.0"/>
